File: hardware/Irrigacao_mesh/Irrigacao_mesh.kicad_sch (KiCad schematic)
At the start: 96 parts, among them J1 USB_5V_IN, J10 IN0, J11 IN1, J12 IN2, J13 IN3, J14 SENSOR0, J15 SENSOR1, J2 12V_BAT, J4 RTC_PCF8563, J5 UART_PROG, J6 VALVE0, J7 VALVE1, J8 RELAY0_OUT, J9 RELAY1_OUT, K1 FINDER-36.11-5V, K2 FINDER-36.11-5V, Q1 MMBT3904, Q2 MMBT3904, SW1 BOOT/USER, U1 ESP32-WROOM-32, U2 AMS1117-3.3, U3 HT-RA62, U4 L298N, U5 LTV-817, U6 LTV-817, U7 LTV-817, U8 LTV-817

Commit message: Update na placa
Parts:
- added TP1, TP2: TestPoint, TestPoint:TestPoint_Pad_D4.0mm, symbol Connector:TestPoint
- R20, R21: footprint Resistor_SMD:R_0805_2012Metric -> Resistor_SMD:R_0603_1608Metric
- SW1: footprint Button_Switch_SMD:SW_SPST_TL3305A -> Button_Switch_SMD:SW_Push_1P1T_XKB_TS-1187A
Connections:
- net +5V: now also TP1.1
- net GND: now also TP2.1

Commit message: Adição de leds no TX e RX
Parts:
- added D20, D22: LED_TX, LED_SMD:LED_0805_2012Metric, symbol Device:LED
- added JP10: SolderJumper_2_Bridged, Jumper:SolderJumper-2_P1.3mm_Bridged_Pad1.0x1.5mm, symbol Jumper:SolderJumper_2_Bridged
- added Q3, Q4: MMBT3904, Package_TO_SOT_SMD:SOT-23, symbol Transistor_BJT:MMBT3904
- added R24, R27: 10k, Resistor_SMD:R_0805_2012Metric, symbol Device:R
- added R25, R26: 470, Resistor_SMD:R_0805_2012Metric, symbol Device:R
- added TP3, TP4: TestPoint, TestPoint:TestPoint_Pad_D4.0mm, symbol Connector:TestPoint
Connections:
- net +12V: now also TP3.1
- net +3V3: now also R25.1, R26.1
- net GND: now also JP10.2 (B), Q3.2 (E), Q4.2 (E)
- net GND1: now also JP10.1 (A), TP4.1
- net REL0_NC: now also J8.3 (Pin_3); no longer J8.1 (Pin_1)
- net REL0_NO: now also J8.1 (Pin_1); no longer J8.3 (Pin_3)
- net REL1_NC: now also J9.3 (Pin_3); no longer J9.1 (Pin_1)
- net REL1_NO: now also J9.1 (Pin_1); no longer J9.3 (Pin_3)
- net UART_RX: now also R27.1
- net UART_TX: now also R24.1
- new net RXLED_A: D22.2 (A), R26.2
- new net RXLED_B: Q4.1 (B), R27.2
- new net RXLED_K: D22.1 (K), Q4.3 (C)
- new net TXLED_A: D20.2 (A), R25.2
- new net TXLED_B: Q3.1 (B), R24.2
- new net TXLED_K: D20.1 (K), Q3.3 (C)
Other:
- moved on the sheet: C10, C11, C12, C9, D11, J9, JP9, U4
